Commit message: second_commit

File: description/ros2_control.xacro (robot description, xacro)
@@ -72,5 +72,5 @@
                 <state_interface name="position"/>
             </joint>
-            <joint name="joint_5">
+            <!-- <joint name="joint_5">
                 <command_interface name="position">
                 <param name="min">-${PI / 2}</param>
@@ -78,5 +78,5 @@
                 </command_interface>
                 <state_interface name="position"/>
-            </joint>
+            </joint>  -->
         </ros2_control>
     </xacro:unless>
