Commit message: 132

File: description/arm_robot.xacro (robot description, xacro)
@@ -181,5 +181,5 @@
         <parent link="hand_1_link" />
         <child link="hand_2_link" />
-        <origin xyz="0 0 ${hand_length}" rpy="0 0 0" />
+        <origin xyz="0 0 ${hand_length}" rpy="0 0 ${pi}" />
         <axis xyz="0 1 0" />
         <limit lower="${-pi/2}" upper="${pi/2}" effort="100" velocity="100" />

File: description/robot.urdf.xacro (robot description, xacro)
@@ -1,7 +1,10 @@
 <?xml version="1.0"?>
-<robot xmlns:xacro="http://www.ros.org/wiki/xacro"  name="articubot">
+<robot xmlns:xacro="http://www.ros.org/wiki/xacro"  name="robot">
     <xacro:arg name="use_ros2_control" default="true"/>
     <xacro:arg name="sim_mode" default="false"/>
     <xacro:include filename="robot_core.xacro" />
+    <xacro:include filename="arm_robot.xacro" />
+    <xacro:include filename="inertial_macros.xacro" />
+    <xacro:include filename="camera.xacro" />
     <xacro:if value="$(arg use_ros2_control)">
         <xacro:include filename="ros2_control.xacro" />
@@ -11,7 +14,4 @@
     </xacro:unless>
     <xacro:include filename="lidar.xacro" />
-    <xacro:include filename="camera.xacro" />
-    <xacro:include filename="arm_robot.xacro" />
-    <xacro:include filename="inertial_macros.xacro" />
     <!-- <xacro:include filename="depth_camera.xacro" /> -->
     <xacro:include filename="face.xacro" />

File: description/ros2_control.xacro (robot description, xacro)
@@ -54,5 +54,5 @@
                 <command_interface name="position">
                 <param name="min">-${PI / 2}</param>
-                <param name="max">0.0</param>
+                <param name="max">${PI / 2}</param>
                 </command_interface>
                 <state_interface name="position"/>
@@ -61,5 +61,5 @@
                 <command_interface name="position">
                 <param name="min">-${PI / 2}</param>
-                <param name="max">0.0</param>
+                <param name="max">${PI / 2}</param>
                 </command_interface>
                 <state_interface name="position"/>
